Commit message: fix camera collider size

File: turtlebot3_description/urdf/turtlebot3_burger.urdf.xacro (robot description, xacro)
@@ -161,5 +161,5 @@
       <origin xyz="0 0 0" rpy="0 0 0"/>
       <geometry>
-        <box size=".01 .01 .01"/>
+        <box size=".02 .02 .02"/>
       </geometry>
     </collision>
